File: Kicad/MiniSumoSTM.kicad_pcb (KiCad board)
At the start: 2 copper layers, 93 x 85.8 mm, 67 parts, among them J10 Conn_01x03_Pin, J2 USB_B_Micro, J4 Conn_02x03_Top_Bottom, M1 Conn_01x02_Pin, M2 Conn_01x02_Pin, Q3 AON7422G, Q4 AON7422G, U1 ITR8307, U11 LD1117S33TR_SOT223, U2 ITR8307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

Commit message: fixed pcb
Parts:
- added R18: 1k5, Resistor_SMD:R_0805_2012Metric_Pad1.20x1.40mm_HandSolder, B.Cu at (171.9, 77.2)
- R7: value 1k5 -> 10k
- moved R7 0.17 mm to (154.1, 77.7)
- renumbered M2 to M1, M1 to M2, TF1 to ToF1
Connections:
- J4 pad 5: /MCU/SWO -> unconnected-(J4-Pin_5-Pad5)
- R7 pad 1: +3.3V -> GND
- R7 pad 2: /MCU/SCL1 -> /MCU/BOOT0
- U4 pad 39: unconnected-(U4-PA15-Pad39) -> /MCU/SCL1
- U4 pad 40: /MCU/SWO -> unconnected-(U4-PB3-Pad40)
- U4 pad 45: /MCU/SCL1 -> /MCU/BOOT0
Routing:
- net /MCU/SWO: track 24.0 -> 0.00 mm, vias 1 -> 0
- net /MCU/BOOT0: track 0.00 -> 10.6 mm, vias 0 -> 1
- net +3.3V: track 342.3 -> 343.4 mm
- net GND: vias 452 -> 450
